File: pcb/revA/mdt-chipdown.kicad_pcb (KiCad board)
At the start: 2 copper layers, 94 x 79.6 mm, 81 parts, among them J1 SPDIF IN, J2 SPDIF OUT, J3 G3, SW1 ON_OFF, SW2 PROGRAM, U1 AMS1117-3.3, U2 Teensy4.1, U3 PCM5102A, U4 ILI9341 3.2" capacitive touch, U5 W25Q128JVS

Commit message: Added logo
Parts:
- added LOGO3: logo, footprints:microDXD_logo12, F.Cu at (85.3, 106.3)
Other:
- board text added: "Chipdown Rev.${REVISION}"
- board text added: "DN"
- board text removed: "DOWN"
- board text removed: "MicroDEXED Touch Chipdown"
- board text removed: "Rev.${REVISION}"
