File: pcb/revA/mdt-chipdown.kicad_sch (KiCad schematic)
At the start: 81 parts, among them J1 SPDIF IN, J2 SPDIF OUT, J3 G3, SW1 ON_OFF, SW2 PROGRAM, U1 AMS1117-3.3, U2 Teensy4.1, U3 PCM5102A, U4 ILI9341 3.2" capacitive touch, U5 W25Q128JVS

Commit message: Added logo
Parts:
- added LOGO3: logo, footprints:microDXD_logo12, symbol my:logo
Changed lines of the file:
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@@
+	)
+	(symbol
+		(lib_id "my:logo")
+		(at 102.87 121.92 0)
+		(unit 1)
+		(body_style 1)
+		(exclude_from_sim no)
+		(in_bom no)
+		(on_board yes)
+		(in_pos_files yes)
+		(dnp no)
+		(fields_autoplaced yes)
+		(property "Reference" "LOGO3"
+			(at 102.87 116.84 0)
+			(hide yes)
+			(show_name no)
+			(do_not_autoplace no)
+			(effects
+				(font
+					(size 1.27 1.27)
+				)
+			)
+		)
+		(property "Value" "logo"
+			(at 102.87 128.27 0)
+			(hide yes)
+			(show_name no)
+			(do_not_autoplace no)
+			(effects
+				(font
+					(size 1.27 1.27)
+				)
+			)
+		)
+		(property "Footprint" "footprints:microDXD_logo12"
+			(at 102.87 127 0)
+			(hide yes)
+			(show_name no)
+			(do_not_autoplace no)
+			(effects
+				(font
+					(size 1.27 1.27)
+				)
+			)
+		)
+		(property "Datasheet" ""
+			(at 103.632 127 0)
+			(hide yes)
+			(show_name no)
+			(do_not_autoplace no)
+			(effects
+				(font
+					(size 1.27 1.27)
+				)
+			)
+		)
+		(property "Description" ""
+			(at 102.87 121.92 0)
+			(hide yes)
+			(show_name no)
+			(do_not_autoplace no)
+			(effects
+				(font
+					(size 1.27 1.27)
+				)
+			)
+		)
+		(instances
+			(project "mdt-chipdown"
+				(path "/8761c4bf-5316-457a-a770-398e72936388"
+					(reference "LOGO3")
+					(unit 1)
+				)
+			)
+		)
 	)
 	(symbol

Commit message: Updated revA: replaced jumpers with solder jumpers (preconfigured)
Parts:
- added JP5, JP6: Jumper_2_Open, Jumper:SolderJumper-2_P1.3mm_Open_RoundedPad1.0x1.5mm, symbol Jumper:Jumper_2_Open
- JP1, JP2, JP3, JP4: footprint Connector_PinHeader_2.54mm:PinHeader_1x03_P2.54mm_Vertical -> Jumper:SolderJumper-3_P1.3mm_Bridged12_RoundedPad1.0x1.5mm
Connections:
- net GND: now also JP5.2 (B), JP6.2 (B); no longer TRS2.R2, TRS2.S, TRS3.R2, TRS3.S
- new net: JP5.1 (A), TRS3.R2, TRS3.S
- new net: JP6.1 (A), TRS2.R2, TRS2.S
Other:
- moved on the sheet: D1, JP1, JP2, JP3, JP4, OC1, R3, R4, R7, R8
