File: pcb/revB/mcu.kicad_sch (KiCad schematic)
At the start: 28 parts, among them J4 Micro_SD_Card, J7 Micro_SD_Card, U2 APS1604M-3SQRx-SN, U6 MKL02Z32VFG4, U7 MIMXRT1062DVJ6B, U8 GD25Q64ESIGR, U9 APS1604M-3SQRx-SN, Y1 24MHz, Y2 32768

Commit message: revB, fully routed
Parts:
- added C29, C31: 100n, Capacitor_SMD:C_0805_2012Metric_Pad1.18x1.45mm_HandSolder, symbol Device:C
- added R16, R17, R18, R19: 10k, Resistor_SMD:R_0805_2012Metric_Pad1.20x1.40mm_HandSolder, symbol Device:R
- added TP8: GPIO_AD_B0_00, TestPoint:TestPoint_Pad_2.0x2.0mm, symbol Connector:TestPoint
- TP1: renamed from TP11; value TestPoint -> GPIO_AD_B1_12
- TP2: renamed from TP10; value TestPoint -> GPIO_AD_B1_13
- TP3: renamed from TP8; value TestPoint -> CV GATE IN
- TP4: renamed from TP9; value TestPoint -> CV CLOCK IN
- TP5: renamed from TP13; value TestPoint -> CV IN
- TP6: renamed from TP14; value TestPoint -> MCP INTA
- TP7: renamed from TP12; value TestPoint -> MEM CS
- U5: renamed from U2; value APS1604M-3SQRx-SN -> APS6404L-3SQR
- U6: renamed from U9; value APS1604M-3SQRx-SN -> APS6404L-3SQR
- renumbered C25 to C22, C26 to C23, C48 to C25, C49 to C26, C23 to C27, C50 to C28, C51 to C30, D6 to D5, J7 to J5, R10 to R13, R17 to R14, R16 to R15, U6 to U7, U7 to U9
Connections:
- net GND: now also J5.SH (SHIELD), C29.2, C31.2
- net SPI_MISO: now also R19.2
- net SPI_MOSI: now also R17.2
- net SPI_SCK: now also R18.2
- net VPP3_3: now also C29.1, C31.1, R16.1, R17.1, R18.1, R19.1
- net ~{SD2_CS}: now also R16.2
- net at U9.M14 (GPIO_AD_B0_00): now also TP8.1
- no-connect marks 17 -> 16
Other:
- note added: "ETH Pins Unused"
- note added: "Warning! The MLK02Z32 MCU should be ordered directly from PJRC (pre-programmed with teensy bootloader!) https://www.pjrc.com/store/ic_mkl02_t4.html"
- note removed: "TODO: TP"
- note removed: "TODO: pullups"
- moved on the sheet: TP3, TP4, TP5, TP6, TP7, U9C

Commit message: Added custom field HighlightPins
Parts:
- J4: HighlightPins (none) -> 1,2,3,5,7,8
- J5: HighlightPins (none) -> 2,3,5,7
- R13: HighlightPins (none) -> 2
- TP1, TP2, TP3, TP4, TP5, TP6, TP7, TP8: HighlightPins (none) -> 1
- U5, U6, U8: HighlightPins (none) -> 1,2,3,5,6,7
- U7: HighlightPins (none) -> 4,5,8,13,7,6,15,12,9,3
- Y1: HighlightPins (none) -> 1,3; private KLC_S4.1 -> KLC_S3.3
- Y2: HighlightPins (none) -> 1,2
Changed lines of the file:
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@@
 			)
 		)
+		(property "HighlightPins" "1,2"
+			(at 133.35 154.94 0)
+			(hide yes)
+			(show_name no)
+			(do_not_autoplace no)
+			(effects
+				(font
+					(size 1.27 1.27)
+				)
+			)
+		)
 		(pin "3"
 		)
@@
 			)
 		)
+		(property "HighlightPins" "1"
+			(at 189.23 139.7 90)
+			(hide yes)
+			(show_name no)
+			(do_not_autoplace no)
+			(effects
+				(font
+					(size 1.27 1.27)
+				)
+			)
+		)
 		(pin "1"
 		)
@@
 			)
 		)
+		(property "HighlightPins" "1,2,3,5,6,7"
+			(at 45.72 52.07 0)
+			(hide yes)
+			(show_name no)
+			(do_not_autoplace no)
+			(effects
+				(font
+					(size 1.27 1.27)
+				)
+			)
+		)
 		(pin "5"
 		)
@@
 			)
 		)
+		(property "HighlightPins" "1"
+			(at 248.92 149.86 90)
+			(hide yes)
+			(show_name no)
+			(do_not_autoplace no)
+			(effects
+				(font
+					(size 1.27 1.27)
+				)
+			)
+		)
 		(pin "1"
 		)
@@
 			)
 		)
+		(property "HighlightPins" "4,5,8,13,7,6,15,12,9,3"
+			(at 107.95 118.11 0)
+			(hide yes)
+			(show_name no)
+			(do_not_autoplace no)
+			(effects
+				(font
+					(size 1.27 1.27)
+				)
+			)
+		)
 		(pin "1"
 		)
@@
 			)
 		)
+		(property "HighlightPins" "1,2,3,5,6,7"
+			(at 111.76 81.28 0)
+			(hide yes)
+			(show_name no)
+			(do_not_autoplace no)
+			(effects
+				(font
+					(size 1.27 1.27)
+				)
+			)
+		)
 		(pin "2"
 		)
@@
 			)
 		)
+		(property "HighlightPins" "2"
+			(at 49.53 121.92 90)
+			(hide yes)
+			(show_name no)
+			(do_not_autoplace no)
+			(effects
+				(font
+					(size 1.27 1.27)
+				)
+			)
+		)
 		(pin "1"
 		)
@@
 			)
 		)
+		(property "HighlightPins" "1"
+			(at 248.92 154.94 90)
+			(hide yes)
+			(show_name no)
+			(do_not_autoplace no)
+			(effects
+				(font
+					(size 1.27 1.27)
+				)
+			)
+		)
 		(pin "1"
 		)
@@
 			)
 		)
+		(property "HighlightPins" "2,3,5,7"
+			(at 240.03 36.83 0)
+			(hide yes)
+			(show_name no)
+			(do_not_autoplace no)
+			(effects
+				(font
+					(size 1.27 1.27)
+				)
+			)
+		)
 		(pin "8"
 		)
@@
 			)
 		)
+		(property "HighlightPins" "1"
+			(at 248.92 152.4 90)
+			(hide yes)
+			(show_name no)
+			(do_not_autoplace no)
+			(effects
+				(font
+					(size 1.27 1.27)
+				)
+			)
+		)
 		(pin "1"
 		)
@@
 			)
 		)
+		(property "HighlightPins" "1"
+			(at 264.16 100.33 90)
+			(hide yes)
+			(show_name no)
+			(do_not_autoplace no)
+			(effects
+				(font
+					(size 1.27 1.27)
+				)
+			)
+		)
 		(pin "1"
 		)
@@
 			)
 		)
+		(property "HighlightPins" "1"
+			(at 248.92 157.48 90)
+			(hide yes)
+			(show_name no)
+			(do_not_autoplace no)
+			(effects
+				(font
+					(size 1.27 1.27)
+				)
+			)
+		)
 		(pin "1"
 		)
@@
 			)
 		)
+		(property "HighlightPins" "1,2,3,5,6,7"
+			(at 45.72 88.9 0)
+			(hide yes)
+			(show_name no)
+			(do_not_autoplace no)
+			(effects
+				(font
+					(size 1.27 1.27)
+				)
+			)
+		)
 		(pin "5"
 		)
@@
 			)
 		)
+		(property "HighlightPins" "1,2,3,5,7,8"
+			(at 100.33 38.1 0)
+			(hide yes)
+			(show_name no)
+			(do_not_autoplace no)
+			(effects
+				(font
+					(size 1.27 1.27)
+				)
+			)
+		)
 		(pin "8"
 		)
@@
 			)
 		)
+		(property "HighlightPins" "1"
+			(at 248.92 147.32 90)
+			(hide yes)
+			(show_name no)
+			(do_not_autoplace no)
+			(effects
+				(font
+					(size 1.27 1.27)
+				)
+			)
+		)
 		(pin "1"
 		)
@@
 			)
 		)
+		(property "HighlightPins" "1"
+			(at 189.23 137.16 90)
+			(hide yes)
+			(show_name no)
+			(do_not_autoplace no)
+			(effects
+				(font
+					(size 1.27 1.27)
+				)
+			)
+		)
 		(pin "1"
 		)
@@
 			)
 		)
-		(property private "KLC_S4.1" "Some pins are on 50mil grid to make the symbol small"
-			(at 85.09 170.18 0)
+		(property "HighlightPins" "1,3"
+			(at 85.09 154.94 0)
 			(hide yes)
-			(show_name yes)
+			(show_name no)
+			(do_not_autoplace no)
+			(effects
+				(font
+					(size 1.27 1.27)
+				)
+			)
+		)
+		(property "Field8" ""
+			(at 85.09 154.94 0)
+			(hide yes)
+			(show_name no)
 			(do_not_autoplace no)
 			(effects
