File: pcb/revB/mcu_power.kicad_sch (KiCad schematic)
At the start: 29 parts, among them Q1 DMG2305UX, U10 TLV75733PDBV, U7 MIMXRT1062DVJ6B

Commit message: revB, fully routed
Parts:
- renumbered C42 to C32, C43 to C33, C40 to C34, C31 to C35, C35 to C36, C27 to C37, C44 to C38, C41 to C39, C32 to C40, C36 to C41, C28 to C42, C38 to C43, C45 to C44, C33 to C45, C37 to C46, C29 to C47, C39 to C48, C46 to C49, C34 to C50, C30 to C51, C47 to C52, D5 to D6, L3 to L1, L1 to L3, R15 to R20, U7 to U9
Connections:
- net PMIC_ON_REQ: now reaches R20.2, U10.3 (EN), U9.K7 (PMIC_ON_REQ)
- net VDD_SNVS_IN: now reaches C32.1, D6.3, U9.M9 (VDD_SNVS_IN)
Other:
- moved on the sheet: C32, C33, C38, C44, C49, C52, L3

Commit message: Updated revB: changed vias from 0.4/0.3 to 0.45/0.2
Parts:
- C37, C42, C47, C51: footprint Capacitor_SMD:C_0805_2012Metric_Pad1.18x1.45mm_HandSolder -> Capacitor_SMD:C_0805_2012Metric
- L3: footprint PCM_Inductor_SMD_AKL:L_0805_2012Metric_Pad1.15x1.40mm_HandSolder -> PCM_Inductor_SMD_AKL:L_0805_2012Metric_Pad1.15x1.40mm
Changed lines of the file:
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@@
 			)
 		)
-		(property "Footprint" "Capacitor_SMD:C_0805_2012Metric_Pad1.18x1.45mm_HandSolder"
+		(property "Footprint" "Capacitor_SMD:C_0805_2012Metric"
 			(at 98.0948 116.84 0)
 			(hide yes)
@@
 			)
 		)
-		(property "Footprint" "Capacitor_SMD:C_0805_2012Metric_Pad1.18x1.45mm_HandSolder"
+		(property "Footprint" "Capacitor_SMD:C_0805_2012Metric"
 			(at 128.5748 116.84 0)
 			(hide yes)
@@
 			)
 		)
-		(property "Footprint" "Capacitor_SMD:C_0805_2012Metric_Pad1.18x1.45mm_HandSolder"
+		(property "Footprint" "Capacitor_SMD:C_0805_2012Metric"
 			(at 118.4148 116.84 0)
 			(hide yes)
@@
 			)
 		)
-		(property "Footprint" "PCM_Inductor_SMD_AKL:L_0805_2012Metric_Pad1.15x1.40mm_HandSolder"
+		(property "Footprint" "PCM_Inductor_SMD_AKL:L_0805_2012Metric_Pad1.15x1.40mm"
 			(at 123.19 99.06 0)
 			(hide yes)
@@
 			)
 		)
-		(property "Footprint" "Capacitor_SMD:C_0805_2012Metric_Pad1.18x1.45mm_HandSolder"
+		(property "Footprint" "Capacitor_SMD:C_0805_2012Metric"
 			(at 108.2548 116.84 0)
 			(hide yes)

Commit message: Added custom field HighlightPins
Parts:
- U10: HighlightPins (none) -> 3
Changed lines of the file:
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@@
+			)
+		)
+		(property "HighlightPins" "3"
+			(at 73.66 50.8 0)
+			(hide yes)
+			(show_name no)
+			(do_not_autoplace no)
+			(effects
+				(font
+					(size 1.27 1.27)
+				)
 			)
 		)
