File: pcb/revB/mdt-chipdown.kicad_sch (KiCad schematic)
At the start: 71 parts, among them J2 SPDIF OUT, J5 BI, J6 BI, SW1 ON_OFF, SW2 PROGRAM, U1 AMS1117-3.3, U3 PCM5102A, U4 ILI9341 3.2" capacitive touch, U5 TPD3S014

Commit message: revB, fully routed
Parts:
- renumbered C20 to C10, C22 to C11, C21 to C12, C10 to C13, C11 to C14, C12 to C15, C13 to C16, C14 to C17, C15 to C18, C16 to C19, C18 to C20, C19 to C21, C9 to C8, C8 to C9, H3 to H2, H2 to H3, H7 to H5, H5 to H6, H8 to H7, H6 to H8, J5 to J1, J6 to J2, J2 to J3, LOGO3 to LOGO1, LOGO1 to LOGO2, LOGO2 to LOGO3, R12 to R10, R13 to R11, R14 to R12, R7 to R5, R8 to R6, R5 to R7, R6 to R8, U5 to U1, U1 to U2, U4 to U3, U3 to U4
Connections:
- net VCC: no longer U1.3 (IN)
- new net USB_VBUS: U1.3 (IN)

Commit message: Added custom field HighlightPins
Parts:
- ENC1, ENC2: HighlightPins (none) -> A,B,S1
- J1, J2: HighlightPins (none) -> 2,3,4,5
- J3, R5, R7, R8: HighlightPins (none) -> 2
- OC1: HighlightPins (none) -> 5
- SW1, SW2: HighlightPins (none) -> 1
- U3: HighlightPins (none) -> 3,4,5,6,7,8,10,11,12,13
- U4: HighlightPins (none) -> 15,14,13,17
Changed lines of the file:
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@@
 			)
 		)
+		(property "HighlightPins" "1"
+			(at 167.64 106.68 0)
+			(hide yes)
+			(show_name no)
+			(do_not_autoplace no)
+			(effects
+				(font
+					(size 1.27 1.27)
+				)
+			)
+		)
 		(pin "1"
 		)
@@
 			)
 		)
+		(property "HighlightPins" "2,3,4,5"
+			(at 264.16 30.48 0)
+			(hide yes)
+			(show_name no)
+			(do_not_autoplace no)
+			(effects
+				(font
+					(size 1.27 1.27)
+				)
+			)
+		)
 		(pin "4"
 		)
@@
 			)
 		)
+		(property "HighlightPins" "2,3,4,5"
+			(at 264.16 45.72 0)
+			(hide yes)
+			(show_name no)
+			(do_not_autoplace no)
+			(effects
+				(font
+					(size 1.27 1.27)
+				)
+			)
+		)
 		(pin "4"
 		)
@@
 			)
 		)
+		(property "HighlightPins" "2"
+			(at 158.75 158.75 90)
+			(hide yes)
+			(show_name no)
+			(do_not_autoplace no)
+			(effects
+				(font
+					(size 1.27 1.27)
+				)
+			)
+		)
 		(pin "1"
 		)
@@
 			)
 		)
+		(property "HighlightPins" "A,B,S1"
+			(at 124.46 130.81 0)
+			(hide yes)
+			(show_name no)
+			(do_not_autoplace no)
+			(effects
+				(font
+					(size 1.27 1.27)
+				)
+			)
+		)
 		(pin "C"
 		)
@@
 			)
 		)
+		(property "HighlightPins" "15,14,13,17"
+			(at 217.17 127 0)
+			(hide yes)
+			(show_name no)
+			(do_not_autoplace no)
+			(effects
+				(font
+					(size 1.27 1.27)
+				)
+			)
+		)
 		(pin "1"
 		)
@@
 			)
 		)
+		(property "HighlightPins" "3,4,5,6,7,8,10,11,12,13"
+			(at 214.63 50.8 0)
+			(hide yes)
+			(show_name no)
+			(do_not_autoplace no)
+			(effects
+				(font
+					(size 1.27 1.27)
+				)
+			)
+		)
 		(pin "11"
 		)
@@
 			)
 		)
+		(property "HighlightPins" "2"
+			(at 264.16 69.85 0)
+			(hide yes)
+			(show_name no)
+			(do_not_autoplace no)
+			(effects
+				(font
+					(size 1.27 1.27)
+				)
+			)
+		)
 		(pin "1"
 		)
@@
 			)
 		)
+		(property "HighlightPins" "2"
+			(at 100.33 49.53 90)
+			(hide yes)
+			(show_name no)
+			(do_not_autoplace no)
+			(effects
+				(font
+					(size 1.27 1.27)
+				)
+			)
+		)
 		(pin "1"
 		)
@@
 			)
 		)
+		(property "HighlightPins" "A,B,S1"
+			(at 124.46 109.22 0)
+			(hide yes)
+			(show_name no)
+			(do_not_autoplace no)
+			(effects
+				(font
+					(size 1.27 1.27)
+				)
+			)
+		)
 		(pin "C"
 		)
@@
 			)
 		)
+		(property "HighlightPins" "2"
+			(at 158.75 168.91 90)
+			(hide yes)
+			(show_name no)
+			(do_not_autoplace no)
+			(effects
+				(font
+					(size 1.27 1.27)
+				)
+			)
+		)
 		(pin "1"
 		)
@@
 			)
 		)
+		(property "HighlightPins" "5"
+			(at 85.09 72.39 0)
+			(hide yes)
+			(show_name no)
+			(do_not_autoplace no)
+			(effects
+				(font
+					(size 1.27 1.27)
+				)
+			)
+		)
 		(pin "4"
 		)
@@
 			(at 167.64 124.46 0)
 			(hide yes)
+			(show_name no)
+			(do_not_autoplace no)
+			(effects
+				(font
+					(size 1.27 1.27)
+				)
+			)
+		)
+		(property "HighlightPins" "1"
+			(at 167.64 124.46 0)
+			(hide yes)

Commit message: updated revB with solder jumpers
Parts:
- added JP5, JP6: Jumper_2_Open, Jumper:SolderJumper-2_P1.3mm_Open_RoundedPad1.0x1.5mm, symbol Jumper:Jumper_2_Open
- JP1, JP2, JP3, JP4: footprint Connector_PinHeader_2.54mm:PinHeader_1x03_P2.54mm_Vertical -> Jumper:SolderJumper-3_P1.3mm_Bridged12_RoundedPad1.0x1.5mm
Connections:
- net GND: now also JP5.2 (B), JP6.2 (B); no longer TRS2.R2, TRS2.S, TRS3.R2, TRS3.S
- new net: JP5.1 (A), TRS2.R2, TRS2.S
- new net: JP6.1 (A), TRS3.R2, TRS3.S
Other:
- moved on the sheet: D1, JP1, JP2, JP3, JP4, OC1, R3, R4, R5, R6
