File: pcb/revB1/mcu.kicad_sch (KiCad schematic)
At the start: 35 parts, among them J4 Micro_SD_Card, J5 Micro_SD_Card, U5 APS6404L-3SQR, U6 APS6404L-3SQR, U7 MKL02Z32VFG4, U8 GD25Q64ESIGR, U9 MIMXRT1062DVJ6B, Y1 24MHz, Y2 32768

Commit message: Added (unverified yet) production files for JLC PCBA
Parts:
- C22, C23, C24, C27, C29, C31: LCSC (none) -> C1711
- C25, C26: LCSC (none) -> C152848
- C28, C30: LCSC (none) -> C1727
- D5: LCSC (none) -> C19188468
- J4, J5: LCSC (none) -> C91145
- R13: LCSC (none) -> C17513
- R14: LCSC (none) -> C26113
- R15: LCSC (none) -> C25611
- R16, R17, R18, R19: LCSC (none) -> C17414
- U5, U6: LCSC (none) -> C5333729
- U7: LCSC (none) -> C2056583
- U8: LCSC (none) -> C2831359
- U9: LCSC (none) -> C3216699
- Y1: LCSC (none) -> C15643
- Y2: LCSC (none) -> C2236
