File: pcb/revB1/mcu_power.kicad_sch (KiCad schematic)
At the start: 29 parts, among them Q1 DMG2305UX, U10 TLV75733PDBV, U9 MIMXRT1062DVJ6B

Commit message: Added (unverified yet) production files for JLC PCBA
Parts:
- C32, C38, C39, C43, C45, C46, C47, C48, C49, C52: LCSC (none) -> C5378
- C33, C40, C41, C42, C44: LCSC (none) -> C1779
- C34, C36: LCSC (none) -> C15850
- C35: LCSC (none) -> C19110
- C37: LCSC (none) -> C1713
- C50, C51: LCSC (none) -> C1710
- D6: LCSC (none) -> C37704
- L1, L2: LCSC (none) -> C5671
- L3: LCSC (none) -> C63166
- Q1: LCSC (none) -> C144153
- R20: LCSC (none) -> C25611
- U10: LCSC (none) -> C485517
- U9: LCSC (none) -> C3216699
