File: pcb/revB1/mcu_power.kicad_sch (KiCad schematic)
At the start: 29 parts, among them Q1 DMG2305UX, U10 TLV75733PDBV, U9 MIMXRT1062DVJ6B

Commit message: Updated revB1
Parts:
- U9: footprint footprints:BGA196C80P14X14_1200X1200X152 -> MIMXRT1062DVJ6B:BGA196C80P14X14_1200X1200X152
Changed lines of the file:
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@@
 			)
 		)
-		(property "Footprint" "footprints:BGA196C80P14X14_1200X1200X152"
+		(property "Footprint" "MIMXRT1062DVJ6B:BGA196C80P14X14_1200X1200X152"
 			(at 141.732 156.972 0)
 			(hide yes)
