File: pcb/revB1/mdt-chipdown.kicad_sch (KiCad schematic)
At the start: 74 parts, among them J1 BI, J2 BI, J3 SPDIF OUT, SW1 ON_OFF, SW2 PROGRAM, U1 TPD3S014, U11 74LVC2G06, U2 AMS1117-3.3, U3 ILI9341 3.2" capacitive touch, U4 PCM5102A

Commit message: Added (unverified yet) production files for JLC PCBA
Parts:
- C1, C14, C17, C18, C20, C4, C6: LCSC (none) -> C15850
- C10: LCSC (none) -> C8649
- C11, C12, C15, C21, C5, C53, C7, C8, C9: LCSC (none) -> C1711
- C13: LCSC (none) -> C19110
- C16, C19: LCSC (none) -> C1728
- C2, C3: LCSC (none) -> C2749
- D1, D7: LCSC (none) -> C7420333
- D2: LCSC (none) -> C511038
- D3: LCSC (none) -> C17683617
- D4: LCSC (none) -> C473837
- ENC1, ENC2: LCSC (none) -> C7435302
- F1, F2: LCSC (none) -> C20812
- J1, J2: LCSC (none) -> C5156614
- J3: LCSC (none) -> C5360898
- OC1: LCSC (none) -> C37658
- R1, R2: LCSC (none) -> C26023
- R10: LCSC (none) -> C17477
- R11, R12, R6: LCSC (none) -> C17710
- R3, R5: LCSC (none) -> C25315
- R4: LCSC (none) -> C17557
- R7, R8, R9: LCSC (none) -> C17513
- SW1, SW2: LCSC (none) -> C125050
- TRS1, TRS2, TRS3: LCSC (none) -> C53447038
- U1: LCSC (none) -> C87384
- U11: LCSC (none) -> C402162
- U2: LCSC (none) -> C41414107
- U3: LCSC (none) -> C124407
- U4: LCSC (none) -> C107671
- USB1: LCSC (none) -> C2346
- USB2: LCSC (none) -> C165948
