File: pcb/revB1/mdt-chipdown.kicad_sch (KiCad schematic)
At the start: 75 parts, among them J1 BI, J2 BI, J3 SPDIF OUT, SW1 ON_OFF, SW2 PROGRAM, U1 TPD3S014, U11 74LVC2G06, U2 AMS1117-3.3, U3 ILI9341 3.2" capacitive touch, U4 PCM5102A

Commit message: Updated revB1
Changed lines of the file:
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@@
+	)
+	(junction
+		(at 107.95 80.01)
+		(diameter 0)
+		(color 0 0 0 0)
 	)
 	(junction
 		(at 57.15 90.17)
-		(diameter 0)
-		(color 0 0 0 0)
-	)
-	(junction
-		(at 107.95 80.01)
 		(diameter 0)
 		(color 0 0 0 0)
@@
 	(wire
 		(pts
+			(xy 66.04 82.55) (xy 74.93 82.55)
+		)
+		(stroke
+			(width 0)
+			(type default)
+		)
+	)
+	(wire
+		(pts
 			(xy 203.2 124.46) (xy 203.2 129.54)
 		)
@@
 	(wire
 		(pts
-			(xy 57.15 90.17) (xy 74.93 90.17)
+			(xy 57.15 90.17) (xy 66.04 90.17)
 		)
 		(stroke
@@
 	(wire
 		(pts
-			(xy 74.93 82.55) (xy 74.93 90.17)
-		)
-		(stroke
+			(xy 66.04 82.55) (xy 66.04 90.17)
+		)
+		(stroke
