File: pcb/revB1/mdt-chipdown.kicad_pcb (KiCad board)
At the start: 4 copper layers, 94 x 79.6 mm, 141 parts, among them J1 BI, J2 BI, J3 SPDIF OUT, J4 Micro_SD_Card, J5 Micro_SD_Card, Q1 DMG2305UX, SW1 ON_OFF, SW2 PROGRAM, U1 TPD3S014, U10 TLV75733PDBV, U11 74LVC2G06, U2 AMS1117-3.3, U3 ILI9341 3.2" capacitive touch, U4 PCM5102A, U5 APS6404L-3SQR, U6 APS6404L-3SQR, U7 MKL02Z32VFG4, U8 GD25Q64ESIGR, U9 MIMXRT1062DVJ6B, Y1 24MHz, Y2 32768

Commit message: Updated revB1
Parts:
- moved C51 4.46 mm to (104.8, 70.1), turned to 90 degrees
Routing:
- net /MCU Power/VDD_SOC_IN: track 22.2 -> 23.8 mm
